Commit message: 카메라 포인트클라우드용 좌표계 변환

File: robot_description/urdf/dsr_combined_fixed3 copy.urdf (robot description, URDF)
Before this commit: robot dsr_m0609_complete, 13 links, 12 joints
Links:
- removed link camera_depth_optical_frame
Joints:
- removed joint camera_depth_optical_joint
- joint camera_mount_joint: origin xyz=-0.05 0 -0.03 rpy=0 -1.5708 0 -> xyz=-0.05 0 -0.03 rpy=3.14159 0 3.14159
