Commit message: 가제보 V1_mimic태그 오류 해결

File: robot_description/urdf/dsr_combined_fixed3.urdf (robot description, URDF)
Before this commit: robot dsr_m0609_complete, 13 links, 12 joints
Joints:
- removed joint rg2_finger_joint2
- added joint rg2_finger_joint2_mimic: type revolute, parent rg2_hand, child rg2_rightfinger, origin xyz=0.105 -0.017 0 rpy=0 0 0, axis 0 0 -1, limit lower=0.0 upper=1.18 effort=10.6 velocity=1.57, mimic joint=rg2_finger_joint1 multiplier=1 offset=0

Commit message: rg2 그리퍼 4 bar linkage

File: robot_description/urdf/dsr_combined_fixed3.urdf (robot description, URDF)
Before this commit: robot dsr_m0609_complete, 13 links, 12 joints
Links:
- removed link rg2_hand
- removed link rg2_leftfinger
- removed link rg2_rightfinger
- added link rg2_hand_link, mass 1.684558; collision mesh filename=package://robot_description/meshes/rg2_new/collision/RG2_Ha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; visual mesh filename=package://robot_description/meshes/rg2_new/visual/RG2_Hand_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
- added link rg2_l_finger_link, mass 0.081; collision mesh filename=package://robot_description/meshes/rg2_new/collision/RG2_Le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; visual mesh filename=package://robot_description/meshes/rg2_new/visual/RG2_LeftF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
- added link rg2_l_moment_arm_link, mass 0.160; collision mesh filename=package://robot_description/meshes/rg2_new/collision/RG2_Le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; visual mesh filename=package://robot_description/meshes/rg2_new/visual/RG2_LeftM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
- added link rg2_l_truss_arm_link, mass 0.065; collision mesh filename=package://robot_description/meshes/rg2_new/collision/RG2_Le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; visual mesh filename=package://robot_description/meshes/rg2_new/visual/RG2_LeftT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
- added link rg2_r_finger_link, mass 0.081; collision mesh filename=package://robot_description/meshes/rg2_new/collision/RG2_Ri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; visual mesh filename=package://robot_description/meshes/rg2_new/visual/RG2_Right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
- added link rg2_r_moment_arm_link, mass 0.160; collision mesh filename=package://robot_description/meshes/rg2_new/collision/RG2_Ri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; visual mesh filename=package://robot_description/meshes/rg2_new/visual/RG2_Right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
- added link rg2_r_truss_arm_link, mass 0.065; collision mesh filename=package://robot_description/meshes/rg2_new/collision/RG2_Ri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; visual mesh filename=package://robot_description/meshes/rg2_new/visual/RG2_Right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
Joints:
- removed joint rg2_finger_joint2_mimic
- added joint rg2_l_finger_2_joint: type revolute, parent rg2_l_moment_arm_link, child rg2_l_finger_link, origin xyz=0.049 0.026 0.000 rpy=0 0 0, axis 0 0 1, limit lower=-1.57 upper=1.57 effort=10.6 velocity=3.14, mimic joint=rg2_finger_joint1 multiplier=-1
- added joint rg2_l_finger_passive_joint: type revolute, parent rg2_hand_link, child rg2_l_truss_arm_link, origin xyz=0.122 0.008 0.010 rpy=0 0 0, axis 0 0 1, limit lower=-1.57 upper=1.57 effort=10.6 velocity=3.14, mimic joint=rg2_finger_joint1 multiplier=1
- added joint rg2_r_finger_1_joint: type revolute, parent rg2_hand_link, child rg2_r_moment_arm_link, origin xyz=0.105 -0.017 0.010 rpy=0 0 0, axis 0 0 1, limit lower=-1.57 upper=1.57 effort=10.6 velocity=3.14, mimic joint=rg2_finger_joint1 multiplier=-1
- added joint rg2_r_finger_2_joint: type revolute, parent rg2_r_moment_arm_link, child rg2_r_finger_link, origin xyz=0.049 -0.026 0.000 rpy=0 0 0, axis 0 0 1, limit lower=-1.57 upper=1.57 effort=10.6 velocity=3.14, mimic joint=rg2_finger_joint1 multiplier=1
- added joint rg2_r_finger_passive_joint: type revolute, parent rg2_hand_link, child rg2_r_truss_arm_link, origin xyz=0.122 -0.008 0.010 rpy=0 0 0, axis 0 0 1, limit lower=-1.57 upper=1.57 effort=10.6 velocity=3.14, mimic joint=rg2_finger_joint1 multiplier=-1
- joint rg2_base_joint: child rg2_hand -> rg2_hand_link
- joint rg2_finger_joint1: child rg2_leftfinger -> rg2_l_moment_arm_link; limit lower=0.0 upper=1.18 effort=10.6 velocity=1.57 -> lower=-0.45 upper=1.57 effort=10.6 velocity=3.14; origin xyz=0.105 0.017 0 rpy=0 0 0 -> xyz=0.105 0.017 0.010 rpy=0 0 0; parent rg2_hand -> rg2_hand_link

Commit message: d435i mesh urdf 적용

File: robot_description/urdf/dsr_combined_fixed3.urdf (robot description, URDF)
Before this commit: robot dsr_m0609_complete, 17 links, 16 joints
Links:
- link camera_base_link: geometry collision box size=0.02505 0.090 0.025; visual mesh filename=package://robot_description/meshes/d435.dae
Joints:
- joint camera_mount_joint: origin xyz=-0.05 0 -0.03 rpy=0 -1.5708 0 -> xyz=-0.05 0 0.01 rpy=0 -1.5708 0
